Commit message: Rename the Dex1-1 hand links and joints to MagicSim's g1_dex1 convention
Links: base_link -> hand_palm_link, LinkA_B -> dex1_fingerA_B_link,
d405_mount/d405_camera -> hand_d405_mount_link/hand_d405_camera_link.
Joints: Joint1_1/Joint2_1 -> dex1_finger_joint_1/_2, fixed finger joints
-> dex1_fingerA_B_joint, D405 joints -> hand_d405_{mount,camera,optical}_joint.
The G1 prefixes "<side>_" (e.g. right_hand_palm_link, right_dex1_finger1_3_link).

- URDF, hand USDs (rebuilt), sphere YAML keys, sphere tools and README updated.
- g1_use_dex1_hand.py renames a G1 with the old names first and repoints every
  path to those prims; frames, joints and drives are unchanged (checked against
  the previous G1: identical world poses of all 18 hand bodies, 60 joints, no
  dangling targets).

Co-Authored-By: Claude Opus 5.5 (1M context) <noreply@anthropic.com>

File: dex1_d405_hand/dex1_1_d405.urdf (robot description, URDF)
Before this commit: robot dex1_1_d405, 10 links, 9 joints
Links:
- removed link Link1_1
- removed link Link1_2
- removed link Link1_3
- removed link Link2_1
- removed link Link2_2
- removed link Link2_3
- removed link base_link
- removed link d405_camera
- removed link d405_mount
- removed link d405_optical_frame
- added link dex1_finger1_1_link, mass 0.01; collision mesh filename=meshes/Link1_1.STL; visual mesh filename=meshes/Link1_1.STL
- added link dex1_finger1_2_link, mass 0.01; collision mesh filename=meshes/Link1_2.STL; visual mesh filename=meshes/Link1_2.STL
- added link dex1_finger1_3_link, mass 0.01; collision mesh filename=meshes/Link1_3.STL; visual mesh filename=meshes/Link1_3.STL
- added link dex1_finger2_1_link, mass 0.01; collision mesh filename=meshes/Link2_1.STL; visual mesh filename=meshes/Link2_1.STL
- added link dex1_finger2_2_link, mass 0.01; collision mesh filename=meshes/Link2_2.STL; visual mesh filename=meshes/Link2_2.STL
- added link dex1_finger2_3_link, mass 0.01; collision mesh filename=meshes/Link2_3.STL; visual mesh filename=meshes/Link2_3.STL
- added link hand_d405_camera_link, mass 0.045; collision mesh filename=meshes/d405.STL; visual mesh filename=meshes/d405.STL
- added link hand_d405_mount_link, mass 0.037; collision mesh filename=meshes/d405_mount_collision.STL; visual mesh filename=meshes/d405_mount.STL
- added link hand_d405_optical_frame
- added link hand_palm_link, mass 0.11; collision mesh filename=meshes/base_link_nocam.STL; visual mesh filename=meshes/base_link_nocam.STL
Joints:
- removed joint Joint1_1
- removed joint Joint1_2
- removed joint Joint1_3
- removed joint Joint2_1
- removed joint Joint2_2
- removed joint Joint2_3
- removed joint base_to_d405_mount
- removed joint d405_mount_to_camera
- removed joint d405_mount_to_optical
- added joint dex1_finger1_2_joint: type fixed, parent dex1_finger1_1_link, child dex1_finger1_2_link, origin xyz=-0.013 0.013 0, axis 0 0 0
- added joint dex1_finger1_3_joint: type fixed, parent dex1_finger1_2_link, child dex1_finger1_3_link, origin xyz=-0.0025165 0.025043 -0.001, axis 0 0 0
- added joint dex1_finger2_2_joint: type fixed, parent dex1_finger2_1_link, child dex1_finger2_2_link, origin xyz=0.013 0.013 0, axis 0 0 0
- added joint dex1_finger2_3_joint: type fixed, parent dex1_finger2_2_link, child dex1_finger2_3_link, origin xyz=0.0025165 0.025043 0.0294, axis 0 0 0
- added joint dex1_finger_joint_1: type prismatic, parent hand_palm_link, child dex1_finger1_1_link, origin xyz=0.04055 0.0593 0.0152, axis -1 0 0, limit lower=-0.02 upper=0.0245 effort=20 velocity=0.2
- added joint dex1_finger_joint_2: type prismatic, parent hand_palm_link, child dex1_finger2_1_link, origin xyz=-0.04055 0.0593 -0.0152, axis 1 0 0, limit lower=-0.02 upper=0.0245 effort=20 velocity=0.2
- added joint hand_d405_camera_joint: type fixed, parent hand_d405_mount_link, child hand_d405_camera_link, origin xyz=0.000000 0.058370 0.029108 rpy=0.523611 0.000000 0.000000
- added joint hand_d405_mount_joint: type fixed, parent hand_palm_link, child hand_d405_mount_link, origin xyz=-0.000100 0.033000 -0.001900 rpy=1.570796 0.000000 3.141593
- added joint hand_d405_optical_joint: type fixed, parent hand_d405_mount_link, child hand_d405_optical_frame, origin xyz=0.000000 0.058370 0.029108 rpy=-0.523611 0.000000 3.141593
